File: matrixctl-v1/matrixctl.kicad_pcb (KiCad board)
At the start: 2 copper layers, 53.3 x 15.2 mm, 24 parts, among them J101 Conn_02x05_Odd_Even, J102 Conn_02x05_Odd_Even, J103 Conn_01x08, J104 USB_B_Micro, U101 IS31FL3738, U102 AP7313-33SR

Commit message: actually it's v1
Other:
- board text added: "matrixctl v1 hunz 2020"
- board text removed: "matrixctl v2 hunz 2020"
Changed lines of the file:
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@@
     )
   )
-  (gr_text "matrixctl v2\nhunz 2020" (at 137.9 106) (layer "F.SilkS")
+  (gr_text "matrixctl v1\nhunz 2020" (at 137.9 106) (layer "F.SilkS")
     (effects (font (size 1 1) (thickness 0.15)))
   )
