File: matrixctl-v1/matrixctl.kicad_pcb (KiCad board)
At the start: 2 copper layers, 53.3 x 15.2 mm, 24 parts, among them J101 Conn_02x05_Odd_Even, J102 Conn_02x05_Odd_Even, J103 Conn_01x08, J104 USB_B_Micro, U101 IS31FL3738, U102 AP7313-33SR

Commit message: 22uF->33uF
Parts:
- C101: value 22u/10V -> 33u/10V
