File: matrixctl-v2/matrixctl.kicad_pcb (KiCad board)
At the start: 2 copper layers, 66.8 x 29.7 mm, 31 parts, among them J1 Conn_01x02, J101 Conn_02x05_Odd_Even, J102 Conn_02x05_Odd_Even, J103 Conn_01x08, J104 USB_B_Micro, U1 AP3428, U101 IS31FL3738, U2 bbc_microbit

Commit message: C1 reduced from 22uF to 10uF to reduce risk of acoustic emmisions
Parts:
- C1: value 22u -> 10u

Commit message: 22uF->33uF
Parts:
- C101: value 22u/10V -> 33u/10V
Changed lines of the file:
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@@
       (effects (font (size 1 1) (thickness 0.15)))
     )
-    (fp_text value "22u/10V" (at 0 2.35 90) (layer "F.Fab")
+    (fp_text value "33u/10V" (at 0 2.35 90) (layer "F.Fab")
       (effects (font (size 1 1) (thickness 0.15)))
     )
