File: matrixctl-v2/matrixctl.kicad_sch (KiCad schematic)
At the start: 31 parts, among them J1 Conn_01x02, J101 Conn_02x05_Odd_Even, J102 Conn_02x05_Odd_Even, J103 Conn_01x08, J104 USB_B_Micro, U1 AP3428, U101 IS31FL3738, U2 bbc_microbit

Commit message: add doc-fields in schematics, add PDFs of schematics
Other:
- company: (none) -> hunz <hunz@mailbox.org>
- title: (none) -> Exposure Notifications LED matrix control
Changed lines of the file:
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@@
   (page 1 1)
   (paper "A4")
+  (title_block
+    (title "Exposure Notifications LED matrix control")
+    (rev "2")
+    (company "hunz <hunz@mailbox.org>")
+  )
   (junction (at 25.4 20.32) (diameter 1.016) (color 0 0 0 0))
   (junction (at 31.75 107.95) (diameter 1.016) (color 0 0 0 0))

Commit message: C1 reduced from 22uF to 10uF to reduce risk of acoustic emmisions
Parts:
- C1: value 22u -> 10u
Changed lines of the file:
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@@
       (effects (font (size 1.27 1.27)) (justify left))
     )
-    (property "Value" "22u" (id 1) (at 44.069 163.709 0)
+    (property "Value" "10u" (id 1) (at 44.069 163.709 0)
       (effects (font (size 1.27 1.27)) (justify left))
     )
@@
     )
     (path "/d1ea1858-ca89-4b7d-8ee8-e728aaa548fb"
-      (reference "C1") (unit 1) (value "22u") (footprint "Capacitor_SMD:C_0805_2012Metric")
+      (reference "C1") (unit 1) (value "10u") (footprint "Capacitor_SMD:C_0805_2012Metric")
     )
     (path "/dcf3bb4f-4c61-41a5-afcc-dfab8c6540a5"

Commit message: 22uF->33uF
Parts:
- C101: value 22u/10V -> 33u/10V
Changed lines of the file:
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@@
       (effects (font (size 1.27 1.27)) (justify right))
     )
-    (property "Value" "22u/10V" (id 1) (at 98.171 25.279 0)
+    (property "Value" "33u/10V" (id 1) (at 98.171 25.279 0)
       (effects (font (size 1.27 1.27)) (justify right))
     )
@@
     )
     (path "/55938adc-8b31-40b2-bf95-6c3e624a32f2"
-      (reference "C101") (unit 1) (value "22u/10V") (footprint "Capacitor_Tantalum_SMD:CP_EIA-3528-21_Kemet-B")
+      (reference "C101") (unit 1) (value "33u/10V") (footprint "Capacitor_Tantalum_SMD:CP_EIA-3528-21_Kemet-B")
     )
     (path "/ef27c1dd-5522-490f-b6dd-9a9950ca1e1d"
